File: docs/projects/tvpong/tvpong.sch (EAGLE design)
At the start: 19 parts, among them IC1 MEGA8-P, Q1 12MHz, X3 AUDIO, X4 VIDEO

Commit message: pong
Parts:
- removed JP4: Reset, jumper:JP1E
- removed LED4: POW USB, led:LED3MM
- removed R8: 1k, rcl:R-EU_0204/5
- removed X1: (no value), con-berg:PN61729
- removed X2: (no value), con-harting-ml:ML10L
- added JP1: (no value), jumper:JP1E
- added S1: (no value), switch-omron:31-XX
- added SV1: ISP, con-lstb:MA06-1
- added SV2: POT1, con-lstb:MA03-1
- added SV3: POT2, con-lstb:MA03-1
- C1: device rcl:CPOL-EUTT2D5 -> rcl:CPOL-EUTT5D7
- Q1: value 12MHz -> 20MHz
- R1: device rcl:R-EU_0207/12 -> rcl:R-EU_0204/5
- R2: device rcl:R-EU_0207/15 -> rcl:R-EU_0204/7
Connections:
- removed net UNUSED: X2.3
- new net N$3: IC1.PC4(ADC4/SDA), SV2.2
- new net N$9: IC1.PD4(XCK/T0), S1.P
- net +5V: now also JP1.1, SV1.3, SV2.1, SV3.1; no longer R8.1, X1.1, X2.2
- net GND: now also JP1.2, S1.S, SV1.1, SV2.3, SV3.3; no longer JP4.2, LED4.C, X1.4, X2.10, X2.4, X2.6, X2.8
- net MISO: now also SV1.5; no longer X2.9
- net MOSI: now also SV1.6; no longer X2.1
- net N$4: now also IC1.PC5(ADC5/SCL), SV3.2; no longer LED4.A, R8.2
- net RST: now also SV1.2; no longer JP4.1, X2.5
- net SCK: now also SV1.4; no longer X2.7
Other:
- moved on the sheet: D1, D2, R1, R2
