File: docs/projects/usb_1wire_hub/usb_1wire_hub.brd (EAGLE design)
At the start: 47.9 x 44.4 mm, 26 parts, among them Q1 12MHz

Commit message: fix airwires
Changed lines of the file:
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@@
 <wire x1="30.48" y1="5.08" x2="20.32" y2="5.08" width="0.4064" layer="16"/>
 <wire x1="30.48" y1="5.08" x2="50.8" y2="5.08" width="0.4064" layer="16"/>
-<wire x1="12.7" y1="27.94" x2="12.33" y2="27.96" width="0" layer="19" extent="16-16"/>
 <via x="25.4" y="27.94" extent="1-16" drill="0.6" shape="square"/>
 <via x="25.4" y="45.72" extent="1-16" drill="0.6" shape="square"/>
 <via x="12.7" y="45.72" extent="1-16" drill="0.6" shape="square"/>
 <via x="12.7" y="5.08" extent="1-16" drill="0.6" shape="square"/>
+<wire x1="12.33" y1="27.96" x2="12.7" y2="27.96" width="0.4064" layer="16"/>
+<wire x1="12.7" y1="27.96" x2="12.7" y2="27.94" width="0.4064" layer="16"/>
 </signal>
 <signal name="N$2">
