File: docs/projects/wire_detector/wire_detector.brd (EAGLE design)
At the start: 25.1 x 27.9 mm, 7 parts, among them IC3 7414N

Commit message: fix airwires
Changed lines of the file:
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@@
 <wire x1="33.02" y1="50.8" x2="33.02" y2="45.72" width="0.4064" layer="16"/>
 <wire x1="38.1" y1="45.72" x2="38.1" y2="50.8" width="0.4064" layer="16"/>
-<wire x1="35.56" y1="30.48" x2="35.56" y2="38.1" width="0.4064" layer="16"/>
+<wire x1="35.56" y1="33.02" x2="35.56" y2="38.1" width="0.4064" layer="16"/>
 <wire x1="30.48" y1="30.48" x2="30.48" y2="38.1" width="0.4064" layer="16"/>
 <wire x1="30.48" y1="30.48" x2="35.56" y2="30.48" width="0.4064" layer="1"/>
@@
 <wire x1="38.1" y1="43.18" x2="38.1" y2="45.72" width="0.4064" layer="16"/>
 <wire x1="35.56" y1="40.64" x2="38.1" y2="43.18" width="0.4064" layer="1"/>
-<wire x1="35.56" y1="30.48" x2="35.56" y2="33.02" width="0" layer="19" extent="16-16"/>
 <via x="27.94" y="50.8" extent="1-16" drill="0.6" shape="square"/>
 <via x="33.02" y="50.8" extent="1-16" drill="0.6" shape="square"/>
@@
 <via x="35.56" y="40.64" extent="1-16" drill="0.6" shape="square"/>
 <via x="38.1" y="43.18" extent="1-16" drill="0.6" shape="square"/>
+<wire x1="35.56" y1="33.02" x2="35.56" y2="30.48" width="0.4064" layer="16"/>
 </signal>
 <signal name="N$3">
@@
 <wire x1="27.94" y1="33.02" x2="27.94" y2="38.1" width="0.4064" layer="16"/>
 <wire x1="33.02" y1="33.02" x2="33.02" y2="38.1" width="0.4064" layer="16"/>
-<wire x1="27.94" y1="30.48" x2="33.02" y2="33.02" width="0" layer="19" extent="1-16"/>
 <wire x1="25.4" y1="30.48" x2="25.4" y2="38.1" width="0.4064" layer="16"/>
 <wire x1="25.4" y1="30.48" x2="27.94" y2="30.48" width="0.4064" layer="1"/>
