File: docs/projects/outlet_tester/outlet_tester.sch (EAGLE design)
At the start: 20 parts

Commit message: outlet tester: adjust to available parts
Parts:
- added R8, R9: 2.2k 3W, rcl:R-EU_0207/10
- R7: value 6.8k 8W -> 2.2k 3W
Connections:
- new net N$10: R8.2, R9.1
- new net N$9: R7.2, R8.1
- net 1: now also R9.2; no longer R7.2
Other:
- note added: "3 mA"
- note added: "30 mA"
- moved on the sheet: 1, 2, GND
Changed lines of the file:
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@@
 <?xml version="1.0" encoding="utf-8"?>
 <!DOCTYPE eagle SYSTEM "eagle.dtd">
-<eagle version="6.2">
+<eagle version="6.4">
 <drawing>
 <settings>
@@
 </part>
 <part name="S1" library="switch-misc" deviceset="DT" device="6"/>
-<part name="R7" library="rcl" deviceset="R-EU_" device="0207/10" value="6.8k 8W"/>
+<part name="R7" library="rcl" deviceset="R-EU_" device="0207/10" value="2.2k 3W"/>
+<part name="R8" library="rcl" deviceset="R-EU_" device="0207/10" value="2.2k 3W"/>
+<part name="R9" library="rcl" deviceset="R-EU_" device="0207/10" value="2.2k 3W"/>
 </parts>
 <sheets>
 <sheet>
 <plain>
+<text x="5.08" y="83.82" size="1.778" layer="91" rot="R180">30 mA</text>
+<text x="147.32" y="157.48" size="1.778" layer="91" rot="R180">3 mA</text>
+<text x="144.78" y="116.84" size="1.778" layer="91" rot="R180">3 mA</text>
+<text x="144.78" y="73.66" size="1.778" layer="91" rot="R180">3 mA</text>
 </plain>
 <instances>
@@
 <instance part="D6" gate="G$1" x="116.84" y="73.66" rot="R90"/>
 <instance part="R6" gate="G$1" x="73.66" y="60.96" rot="MR180"/>
-<instance part="1" gate="G$1" x="30.48" y="152.4" rot="R270"/>
-<instance part="2" gate="G$1" x="30.48" y="139.7" rot="R270"/>
-<instance part="GND" gate="G$1" x="30.48" y="127" rot="R270"/>
+<instance part="1" gate="G$1" x="-7.62" y="165.1" rot="R270"/>
+<instance part="2" gate="G$1" x="-7.62" y="152.4" rot="R270"/>
+<instance part="GND" gate="G$1" x="-7.62" y="139.7" rot="R270"/>
 <instance part="S1" gate="1" x="17.78" y="83.82"/>
 <instance part="R7" gate="G$1" x="20.32" y="101.6" rot="MR90"/>
+<instance part="R8" gate="G$1" x="20.32" y="114.3" rot="MR90"/>
+<instance part="R9" gate="G$1" x="20.32" y="127" rot="MR90"/>
 </instances>
 <busses>
@@
 </segment>
 <segment>
-<wire x1="27.94" y1="127" x2="20.32" y2="127" width="0.1524" layer="91"/>
-<label x="20.32" y="127" size="1.778" layer="95" rot="R180" xref="yes"/>
+<wire x1="-10.16" y1="139.7" x2="-17.78" y2="139.7" width="0.1524" layer="91"/>
+<label x="-17.78" y="139.7" size="1.778" layer="95" rot="R180" xref="yes"/>
 <pinref part="GND" gate="G$1" pin="TP"/>
 </segment>
@@
 </segment>
 <segment>
+<pinref part="R9" gate="G$1" pin="2"/>
+<wire x1="20.32" y1="132.08" x2="20.32" y2="137.16" width="0.1524" layer="91"/>
+<label x="20.32" y="137.16" size="1.778" layer="95" rot="R90" xref="yes"/>
+</segment>
+<segment>
 <pinref part="1" gate="G$1" pin="TP"/>
-<wire x1="27.94" y1="152.4" x2="17.78" y2="152.4" width="0.1524" layer="91"/>
-<label x="17.78" y="152.4" size="1.778" layer="95" rot="R180" xref="yes"/>
-<wire x1="20.32" y1="111.76" x2="20.32" y2="106.68" width="0.1524" layer="91"/>
-<pinref part="R7" gate="G$1" pin="2"/>
-<label x="20.32" y="111.76" size="1.778" layer="95" rot="R90" xref="yes"/>
+<wire x1="-10.16" y1="165.1" x2="-20.32" y2="165.1" width="0.1524" layer="91"/>
+<label x="-20.32" y="165.1" size="1.778" layer="95" rot="R180" xref="yes"/>
 </segment>
 </net>
@@
 </segment>
 <segment>
-<wire x1="27.94" y1="139.7" x2="17.78" y2="139.7" width="0.1524" layer="91"/>
-<label x="17.78" y="139.7" size="1.778" layer="95" rot="R180" xref="yes"/>
+<wire x1="-10.16" y1="152.4" x2="-20.32" y2="152.4" width="0.1524" layer="91"/>
+<label x="-20.32" y="152.4" size="1.778" layer="95" rot="R180" xref="yes"/>
 <pinref part="2" gate="G$1" pin="TP"/>
 </segment>
@@
 </segment>
 </net>
+<net name="N$9" class="0">
+<segment>
+<pinref part="R7" gate="G$1" pin="2"/>
+<pinref part="R8" gate="G$1" pin="1"/>
+<wire x1="20.32" y1="109.22" x2="20.32" y2="106.68" width="0.1524" layer="91"/>
+</segment>
+</net>
+<net name="N$10" class="0">
+<segment>
+<pinref part="R8" gate="G$1" pin="2"/>
+<pinref part="R9" gate="G$1" pin="1"/>
+<wire x1="20.32" y1="121.92" x2="20.32" y2="119.38" width="0.1524" layer="91"/>
+</segment>
+</net>
