File: docs/projects/car_battery_check/car_battery_check.brd (EAGLE design)
At the start: 98.7 x 48.2 mm, 18 parts, among them IC1 7805T, IC2 MEGA8-P

Commit message: carbattery: adding voltage reference (MC1541)
Parts:
- added C2: 1u, rcl:E2,5-6E
- added IC3: MC1541TO, microchip:TO92
- R2: value 22k -> 4k7
- moved R2 2.54 mm to (35.6, 76.2)
Connections:
- net A4: now also C2.+, IC3.2
- net GND: now also C2.-, IC3.1
- net VCC: now also IC3.3
Routing:
- net A4: track 0.00 -> 65.4 mm, vias 0 -> 2
- net GND: track 72.2 -> 125.3 mm, vias 4 -> 6
- net N$1: track 45.5 -> 48.3 mm
- net A5: track 20.1 -> 17.5 mm
- net VCC: track 111.8 -> 113.0 mm
Changed lines of the file:
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@@
 <?xml version="1.0" encoding="utf-8"?>
 <!DOCTYPE eagle SYSTEM "eagle.dtd">
-<eagle version="6.2">
+<eagle version="6.4">
 <drawing>
 <settings>
@@
 </class>
 </classes>
-<designrules>
+<designrules name="default">
 <description language="de">&lt;b&gt;EAGLE Design Rules&lt;/b&gt;
 &lt;p&gt;
@@
 <element name="IC1" library="linear" package="TO220H" value="7805T" x="20.32" y="63.5"/>
 <element name="JP2" library="jumper" package="JP1" value="12V" x="19.05" y="43.18" rot="R90"/>
-<element name="R2" library="rcl" package="R2512" value="22k" x="33.02" y="76.2"/>
+<element name="R2" library="rcl" package="R2512" value="4k7" x="35.56" y="76.2"/>
 <element name="R3" library="rcl" package="0207/15" value="1k" x="48.26" y="63.5"/>
 <element name="C1" library="rcl" package="C025-024X044" value="100n" x="19.05" y="45.72"/>
@@
 <element name="R10" library="rcl" package="0204/7" value="470" x="77.47" y="66.04" rot="R180"/>
 <element name="R11" library="rcl" package="0204/7" value="470" x="48.26" y="46.99" rot="R90"/>
+<element name="IC3" library="microchip" package="TO92" value="MC1541TO" x="25.4" y="50.8" rot="R180">
+<attribute name="OC_NEWARK" value="unknown" x="25.4" y="50.8" size="1.778" layer="27" rot="R180" display="off"/>
+<attribute name="MPN" value="" x="25.4" y="50.8" size="1.778" layer="27" rot="R180" display="off"/>
+<attribute name="MF" value="" x="25.4" y="50.8" size="1.778" layer="27" rot="R180" display="off"/>
+<attribute name="OC_FARNELL" value="unknown" x="25.4" y="50.8" size="1.778" layer="27" rot="R180" display="off"/>
+</element>
+<element name="C2" library="rcl" package="E2,5-6E" value="1u" x="26.67" y="55.88"/>
 </elements>
 <signals>
@@
 <wire x1="20.32" y1="43.18" x2="20.32" y2="45.72" width="0.4064" layer="16"/>
 <wire x1="20.32" y1="45.72" x2="20.32" y2="48.26" width="0.4064" layer="16"/>
-<wire x1="20.32" y1="48.26" x2="58.42" y2="48.26" width="0.4064" layer="1"/>
 <contactref element="C1" pad="2"/>
+<contactref element="IC3" pad="1"/>
+<contactref element="C2" pad="-"/>
+<wire x1="20.32" y1="48.26" x2="21.59" y2="46.99" width="0.4064" layer="1"/>
+<wire x1="21.59" y1="46.99" x2="57.15" y2="46.99" width="0.4064" layer="1"/>
+<wire x1="57.15" y1="46.99" x2="58.42" y2="48.26" width="0.4064" layer="1"/>
+<wire x1="20.32" y1="53.34" x2="20.32" y2="73.66" width="0.4064" layer="16"/>
+<via x="20.32" y="73.66" extent="1-16" drill="0.6" shape="square"/>
+<wire x1="20.32" y1="73.66" x2="27.94" y2="73.66" width="0.4064" layer="1"/>
+<via x="27.94" y="73.66" extent="1-16" drill="0.6" shape="square"/>
+<wire x1="27.94" y1="73.66" x2="27.94" y2="55.88" width="0.4064" layer="16"/>
+<wire x1="27.94" y1="55.88" x2="27.94" y2="50.8" width="0.4064" layer="16"/>
+<wire x1="26.67" y1="50.8" x2="27.94" y2="50.8" width="0.4064" layer="16"/>
 </signal>
 <signal name="VCC">
@@
 <wire x1="55.88" y1="45.72" x2="22.86" y2="45.72" width="0.4064" layer="1"/>
 <via x="22.86" y="45.72" extent="1-16" drill="0.6" shape="square"/>
-<wire x1="22.86" y1="45.72" x2="22.86" y2="53.34" width="0.4064" layer="16"/>
+<wire x1="22.86" y1="45.72" x2="22.86" y2="50.8" width="0.4064" layer="16"/>
+<wire x1="22.86" y1="50.8" x2="22.86" y2="53.34" width="0.4064" layer="16"/>
 <wire x1="60.96" y1="66.04" x2="22.86" y2="66.04" width="0.4064" layer="1"/>
 <via x="22.86" y="66.04" extent="1-16" drill="0.6" shape="square"/>
@@
 <wire x1="22.86" y1="43.18" x2="22.86" y2="45.72" width="0.4064" layer="16"/>
 <wire x1="55.88" y1="45.72" x2="55.88" y2="50.8" width="0.4064" layer="16"/>
+<contactref element="IC3" pad="3"/>
+<wire x1="24.13" y1="50.8" x2="22.86" y2="50.8" width="0.4064" layer="16"/>
 </signal>
 <signal name="N$17">
@@
 <wire x1="58.42" y1="68.58" x2="63.5" y2="68.58" width="0.4064" layer="1"/>
 <wire x1="63.5" y1="68.58" x2="64.77" y2="67.31" width="0.4064" layer="1"/>
-<wire x1="64.77" y1="67.31" x2="64.77" y2="64.77" width="0.4064" layer="1"/>
-<wire x1="64.77" y1="64.77" x2="36.83" y2="64.77" width="0.4064" layer="1"/>
-<wire x1="36.83" y1="64.77" x2="36.83" y2="52.07" width="0.4064" layer="1"/>
+<wire x1="64.77" y1="67.31" x2="64.77" y2="62.23" width="0.4064" layer="1"/>
+<wire x1="64.77" y1="62.23" x2="36.83" y2="62.23" width="0.4064" layer="1"/>
+<wire x1="36.83" y1="62.23" x2="36.83" y2="52.07" width="0.4064" layer="1"/>
 <wire x1="36.83" y1="52.07" x2="40.64" y2="50.8" width="0.4064" layer="1"/>
 <wire x1="40.64" y1="43.18" x2="40.64" y2="50.8" width="0.4064" layer="16"/>
@@
 <wire x1="17.78" y1="76.2" x2="17.78" y2="53.34" width="0.4064" layer="16"/>
 <via x="17.78" y="76.2" extent="1-16" drill="0.6" shape="square"/>
-<wire x1="30.22" y1="76.2" x2="17.78" y2="76.2" width="0.4064" layer="1"/>
 <contactref element="C1" pad="1"/>
+<wire x1="32.76" y1="76.2" x2="32.76" y2="75.94" width="0.4064" layer="1"/>
+<wire x1="32.76" y1="75.94" x2="31.75" y2="76.2" width="0.4064" layer="1"/>
+<wire x1="31.75" y1="76.2" x2="17.78" y2="76.2" width="0.4064" layer="1"/>
 </signal>
 <signal name="A5">
@@
 <wire x1="40.64" y1="63.5" x2="40.64" y2="76.2" width="0.4064" layer="16"/>
 <via x="40.64" y="76.2" extent="1-16" drill="0.6" shape="square"/>
-<wire x1="35.82" y1="76.2" x2="40.64" y2="76.2" width="0.4064" layer="1"/>
+<wire x1="38.36" y1="76.2" x2="40.64" y2="76.2" width="0.4064" layer="1"/>
 </signal>
 <signal name="N$2">
@@
 <signal name="A4">
 <contactref element="IC2" pad="27"/>
+<contactref element="IC3" pad="2"/>
+<contactref element="C2" pad="+"/>
+<wire x1="25.4" y1="55.88" x2="25.4" y2="71.12" width="0.4064" layer="16"/>
+<wire x1="25.4" y1="71.12" x2="25.4" y2="48.895" width="0.4064" layer="16"/>
+<wire x1="43.18" y1="60.96" x2="43.18" y2="71.12" width="0.4064" layer="16"/>
+<via x="43.18" y="71.12" extent="1-16" drill="0.6" shape="square"/>
+<wire x1="43.18" y1="71.12" x2="25.4" y2="71.12" width="0.4064" layer="1"/>
+<via x="25.4" y="71.12" extent="1-16" drill="0.6" shape="square"/>
 </signal>
 </signals>
